Commit message: kinect was added to urdf

File: surenav_description/urdf/surenav_ll.urdf (robot description, URDF)
Before this commit: robot surenav_ll, 13 links, 12 joints
Links:
- added link camera_depth_frame, mass 0.001
- added link camera_depth_optical_frame, mass 0.001
- added link camera_link, mass 0.001; collision box size=0.07271 0.27794 0.073; visual mesh filename=package://surenav_description/meshes/kinect.dae
- added link camera_rgb_frame, mass 0.001
- added link camera_rgb_optical_frame, mass 0.001
- added link world
Joints:
- added joint camera_depth_joint: type fixed, parent camera_rgb_frame, child camera_depth_frame, origin xyz=0 0.0 0 rpy=0 0 0
- added joint camera_depth_optical_joint: type fixed, parent camera_depth_frame, child camera_depth_optical_frame, origin xyz=0 0 0 rpy=-1.57079632679 0 -1.57079632679
- added joint camera_joint: type fixed, parent camera_rgb_frame, child camera_link, origin xyz=-0.031 -0.0 -0.016 rpy=0 0 0
- added joint camera_rgb_joint: type fixed, parent base_link, child camera_rgb_frame, origin xyz=0.16 0 0.48 rpy=0 0 0
- added joint camera_rgb_optical_joint: type fixed, parent camera_rgb_frame, child camera_rgb_optical_frame, origin xyz=0 0 0 rpy=-1.57079632679 0 -1.57079632679
- added joint fixed: type fixed, parent world, child base_link, origin xyz=0.0 -0.0 0.9 rpy=0 0 0

Commit message: surenav_ll control pkg was added.

File: surenav_description/urdf/surenav_ll.urdf (robot description, URDF)
Before this commit: robot surenav_ll, 19 links, 18 joints
Links:
- removed link world
- link l_ankle_roll_link: geometry collision mesh filename=package://surenav_description/meshes/l_ankle_roll_link.dae; visual mesh filename=package://surenav_description/meshes/l_ankle_roll_link.dae
- link r_ankle_roll_link: geometry collision mesh filename=package://surenav_description/meshes/r_ankle_roll_link.dae; visual mesh filename=package://surenav_description/meshes/r_ankle_roll_link.dae
Joints:
- removed joint fixed
- joint camera_rgb_joint: origin xyz=0.16 0 0.48 rpy=0 0 0 -> xyz=0.16 0 1.4 rpy=0 0 0
- joint l_hip_yaw_joint: origin xyz=0.016506 0.1 -0.026 rpy=0 0 0 -> xyz=0.016506 0.1 0.894 rpy=0 0 0
- joint r_hip_yaw_joint: origin xyz=0.016506 -0.1 -0.026 rpy=0 0 0 -> xyz=0.016506 -0.1 0.894 rpy=0 0 0
